Commit message: publish base_scan to scan

File: turtlebot3_description/urdf/turtlebot3_burger.urdf.xacro (robot description, xacro)
@@ -140,3 +140,9 @@
     </inertial>
   </link>
+  <joint name="laser_joint" type="fixed">
+    <parent link="base_scan"/>
+    <child link="laser"/>
+    <origin xyz="0 0 0" rpy="0 0 3.14159"/>
+  </joint>
+  <link name="laser"/>
 </robot>

Commit message: test with livox mid360

File: turtlebot3_description/urdf/turtlebot3_burger.urdf.xacro (robot description, xacro)
@@ -142,7 +142,7 @@
   <joint name="laser_joint" type="fixed">
     <parent link="base_scan"/>
-    <child link="laser"/>
-    <origin xyz="0 0 0" rpy="0 0 3.14159"/>
+    <child link="livox_frame"/>
+    <origin xyz="0 0 0" rpy="0 0 0"/>
   </joint>
-  <link name="laser"/>
+  <link name="livox_frame"/>
 </robot>
